File: hardware/comu.kicad_pcb (KiCad board)
At the start: 2 copper layers, 9.4 x 9 mm, 19 parts, among them J1 USB_A_Embedded, U1 CH32V203F8U6, U2 XC6206PxxxMR

Commit message: Update
Parts:
- D1, D2: footprint Diode_SMD:D_0402_1005Metric -> LED_SMD:LED_0402_1005Metric
- moved TP1 0.13 mm to (147.6, 44.8)
- moved TP5 0.10 mm to (142.0, 45.2)
- moved TP6 0.07 mm to (142.5, 46.0)
Routing:
- net /CAP1B: vias 3 -> 1
- net /CAP1A: vias 3 -> 1
- net /CAP0B: vias 3 -> 1
- net /CAP0A: vias 3 -> 1
Changed lines of the file:
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@@
 		(capping no)
 		(filling no)
+		(aux_axis_origin 145 52.025)
+		(grid_origin 145 52.025)
 		(pcbplotparams
-			(layerselection 0x00000000_00000000_55555555_5755f5ff)
+			(layerselection 0x00000000_00000000_55555555_555555f0)
 			(plot_on_all_layers_selection 0x00000000_00000000_00000000_00000000)
 			(disableapertmacros no)
@@
 			(pdf_single_document no)
 			(dxfpolygonmode yes)
-			(dxfimperialunits yes)
+			(dxfimperialunits no)
 			(dxfusepcbnewfont yes)
 			(psnegative no)
@@
 			(crossoutdnponfab yes)
 			(subtractmaskfromsilk no)
-			(outputformat 1)
+			(outputformat 3)
 			(mirror no)
-			(drillshape 1)
+			(drillshape 0)
 			(scaleselection 1)
 			(outputdirectory "")
@@
 	(footprint "ch32:TestPoint_Pad_D0.6mm"
 		(layer "F.Cu")
-		(at 141.925 45.2)
+		(at 142.02 45.21)
 		(descr "SMD pad as test Point, diameter 1.0mm")
 		(tags "test point SMD pad")
@@
 	(footprint "ch32:TestPoint_Pad_D0.6mm"
 		(layer "F.Cu")
-		(at 147.7 44.7)
+		(at 147.58 44.75)
 		(descr "SMD pad as test Point, diameter 1.0mm")
 		(tags "test point SMD pad")
@@
 	(footprint "ch32:TestPoint_Pad_D0.6mm"
 		(layer "F.Cu")
-		(at 142.39 45.98)
+		(at 142.46 46)
 		(descr "SMD pad as test Point, diameter 1.0mm")
 		(tags "test point SMD pad")
@@
 		(embedded_fonts no)
 	)
-	(footprint "Diode_SMD:D_0402_1005Metric"
+	(footprint "LED_SMD:LED_0402_1005Metric"
 		(layer "F.Cu")
 		(at 141.9 42.6 180)
-		(descr "Diode SMD 0402 (1005 Metric), square (rectangular) end terminal, IPC-7351 nominal, (Body size source: http://www.tortai-tech.com/upload/download/2011102023233369053.pdf)")
-		(tags "diode")
+		(descr "LED SMD 0402 (1005 Metric), square (rectangular) end terminal, IPC-7351 nominal, (Body size source: http://www.tortai-tech.com/upload/download/2011102023233369053.pdf)")
+		(tags "LED")
 		(property "Reference" "D2"
-			(at 0 -1.17 0)
+			(at 0 -1.17 180)
 			(layer "F.SilkS")
 			(hide yes)
@@
 		)
 		(property "Value" "LED"
-			(at 0 1.17 0)
+			(at 0 1.17 180)
 			(layer "F.Fab")
 			(effects
@@
 		)
 		(property "Datasheet" ""
-			(at 0 0 0)
+			(at 0 0 180)
 			(layer "F.Fab")
 			(hide yes)
@@
 		)
 		(property "Description" "Light emitting diode"
-			(at 0 0 0)
+			(at 0 0 180)
 			(layer "F.Fab")
 			(hide yes)
@@
 		)
 		(property "KiLib_Generator" "SMD_2terminal_chip_molded"
-			(at 0 0 0)
+			(at 0 0 180)
 			(layer "F.SilkS")
 			(hide yes)
@@
 		)
 		(fp_text user "${REFERENCE}"
-			(at 0 0 0)
+			(at 0 0 180)
 			(layer "F.Fab")
 			(effects
@@
 		)
 		(embedded_fonts no)
-		(model "${KICAD10_3DMODEL_DIR}/Diode_SMD.3dshapes/D_0402_1005Metric.step"
+		(model "${KICAD10_3DMODEL_DIR}/LED_SMD.3dshapes/LED_0402_1005Metric.step"
 			(offset
 				(xyz 0 0 0)
@@
 		)
 		(embedded_fonts no)
-		(model "${KICAD10_3DMODEL_DIR}/Package_DFN_QFN.3dshapes/QFN-20-1EP_3x3mm_P0.4mm_EP1.65x1.65mm.step"
+		(model "${KICAD10_3DMODEL_DIR}/Package_DFN_QFN.3dshapes/UQFN-20-1EP_3x3mm_P0.4mm_EP1.85x1.85mm.step"
 			(offset
 				(xyz 0 0 0)
@@
 			)
 			(rotate
-				(xyz 0 0 0)
+				(xyz -0 -0 -0)
 			)
 		)
@@
 		(embedded_fonts no)
 	)
-	(footprint "Diode_SMD:D_0402_1005Metric"
+	(footprint "LED_SMD:LED_0402_1005Metric"
 		(layer "F.Cu")
 		(at 148.1 42.6)
-		(descr "Diode SMD 0402 (1005 Metric), square (rectangular) end terminal, IPC-7351 nominal, (Body size source: http://www.tortai-tech.com/upload/download/2011102023233369053.pdf)")
-		(tags "diode")
+		(descr "LED SMD 0402 (1005 Metric), square (rectangular) end terminal, IPC-7351 nominal, (Body size source: http://www.tortai-tech.com/upload/download/2011102023233369053.pdf)")
+		(tags "LED")
 		(property "Reference" "D1"
 			(at 0 -1.17 0)
@@
 		)
 		(embedded_fonts no)
-		(model "${KICAD10_3DMODEL_DIR}/Diode_SMD.3dshapes/D_0402_1005Metric.step"
+		(model "${KICAD10_3DMODEL_DIR}/LED_SMD.3dshapes/LED_0402_1005Metric.step"
 			(offset
 				(xyz 0 0 0)
@@
 		)
 		(property "Value" "Button solder mask removal"
-			(at 0 0.5 90)
+			(at 0 0.5 180)
 			(layer "B.Fab")
 			(effects
@@
 	)
 	(gr_text "B15"
-		(at 141.8 45.2 180)
+		(at 141.81 45.21 180)
 		(layer "F.SilkS")
 		(effects
@@
 	)
 	(gr_text "A8"
-		(at 142 46.05 180)
+		(at 142.07 46.07 180)
 		(layer "F.SilkS")
 		(effects
@@
 	)
 	(gr_text "A3"
-		(at 148 44.7 180)
+		(at 147.88 44.75 180)
 		(layer "F.SilkS")
 		(effects
@@
 	)
 	(via
-		(at 148.5 44.5)
+		(at 148.113131 44.196363)
 		(size 0.6)
 		(drill 0.3)
@@
 	)
 	(segment
-		(start 143.54 45.665)
-		(end 142.865 45.665)
+		(start 142.64 45.4)
+		(end 142.125 45.4)
 		(width 0.2)
 		(layer "F.Cu")
@@
 	)
 	(segment
-		(start 142.865 45.665)
-		(end 142.6 45.4)
+		(start 143.54 45.665)
+		(end 142.905 45.665)
 		(width 0.2)
 		(layer "F.Cu")
@@
 	)
 	(segment
-		(start 142.125 45.4)
-		(end 141.925 45.2)
+		(start 142.905 45.665)
+		(end 142.64 45.4)
 		(width 0.2)
 		(layer "F.Cu")
@@
 	)
 	(segment
-		(start 142.6 45.4)
-		(end 142.125 45.4)
+		(start 142.125 45.4)
+		(end 141.925 45.2)
 		(width 0.2)
 		(layer "F.Cu")
@@
 	)
 	(via
-		(at 149.25 39.85)
-		(size 0.6)
-		(drill 0.3)
-		(layers "F.Cu" "B.Cu")
-		(free yes)
-		(net "/CAP0B")
-	)
-	(via
-		(at 148.6 39.7)
-		(size 0.6)
-		(drill 0.3)
-		(layers "F.Cu" "B.Cu")
-		(free yes)
-		(net "/CAP0B")
-	)
-	(via
-		(at 147.9 39.65)
+		(at 148.2 41.1)
 		(size 0.6)
 		(drill 0.3)
@@
 	)
 	(via
-		(at 146.9 39.5)
-		(size 0.6)
-		(drill 0.3)
-		(layers "F.Cu" "B.Cu")
-		(capping no)
-		(covering
-			(front no)
-			(back no)
-		)
-		(plugging
-			(front no)
-			(back no)
-		)
-		(filling no)
-		(net "/CAP0A")
-	)
-	(via
-		(at 146.25 39.4)
-		(size 0.6)
-		(drill 0.3)
-		(layers "F.Cu" "B.Cu")
-		(capping no)
-		(covering
-			(front no)
-			(back no)
-		)
-		(plugging
-			(front no)
-			(back no)
-		)
-		(filling no)
-		(net "/CAP0A")
-	)
-	(via
-		(at 145.6 39.35)
+		(at 146.93 40.4)
 		(size 0.6)
 		(drill 0.3)
@@
 	)
 	(via
-		(at 144.4 39.35)
-		(size 0.6)
-		(drill 0.3)
-		(layers "F.Cu" "B.Cu")
-		(capping no)
-		(covering
-			(front no)
-			(back no)
-		)
-		(plugging
-			(front no)
-			(back no)
-		)
-		(filling no)
-		(net "/CAP1B")
-	)
-	(via
-		(at 143.1 39.5)
-		(size 0.6)
-		(drill 0.3)
-		(layers "F.Cu" "B.Cu")
-		(capping no)
-		(covering
-			(front no)
-			(back no)
-		)
-		(plugging
-			(front no)
-			(back no)
-		)
-		(filling no)
-		(net "/CAP1B")
-	)
-	(via
-		(at 143.75 39.4)
+		(at 143.1 40.4)
 		(size 0.6)
 		(drill 0.3)
@@
 	)
 	(via
-		(at 142.1 39.55)
-		(size 0.6)
-		(drill 0.3)
-		(layers "F.Cu" "B.Cu")
-		(capping no)
-		(covering
-			(front no)
-			(back no)
-		)
-		(plugging
-			(front no)
-			(back no)
-		)
-		(filling no)
-		(net "/CAP1A")
-	)
-	(via
-		(at 141.4 39.65)
-		(size 0.6)
-		(drill 0.3)
-		(layers "F.Cu" "B.Cu")
-		(capping no)
-		(covering
-			(front no)
-			(back no)
-		)
-		(plugging
-			(front no)
-			(back no)
-		)
-		(filling no)
-		(net "/CAP1A")
-	)
-	(via
-		(at 140.7 39.8)
+		(at 141.9 41.1)
 		(size 0.6)
 		(drill 0.3)
