File: hardware/comu.kicad_sch (KiCad schematic)
At the start: 18 parts, among them J1 USB_A_Embedded, U1 CH32V203F8U6, U2 XC6206PxxxMR

Commit message: Update
Parts:
- D1, D2: footprint Diode_SMD:D_0402_1005Metric -> LED_SMD:LED_0402_1005Metric
- U2: LCSC Part # C5446 -> C51886221
